Commit message: updates

File: src/gazros_test/models/diff_drive_model/diff_drive_model.urdf (robot description, URDF)
Before this commit: robot diff_drive_model, 7 links, 6 joints
Links:
- link sens_ir_fwd_link: geometry collision box size=0.01 0.01 0.01; visual box size=0.01 0.01 0.01

Commit message: Some updates. Program compiles and runs, robot only wants to turn left?

File: src/gazros_test/models/diff_drive_model/diff_drive_model.urdf (robot description, URDF)
Before this commit: robot diff_drive_model, 7 links, 6 joints
Joints:
- joint sens_ir_left_joint: origin xyz=-0.02 0.0178 0 rpy=0 0 1.5707 -> xyz=-0.02 0.0178 -0.01 rpy=0 0 1.5707
- joint sens_ir_right_joint: origin xyz=0.0175 0.0178 0 rpy=0 0 1.5707 -> xyz=0.0175 0.0178 -0.01 rpy=0 0 1.5707
